File: kicad/Audio Jack.kicad_pcb (KiCad board)
At the start: 2 copper layers, 32 x 25.5 mm, 16 parts, among them CN1 PJ-320A, SW1 SW_Push, SW2 SW_Push, SW3 SW_Push, U1 TLV320DAC3100IRHBR

Commit message: Add files via upload
Connections:
- CN1 pad 2: Net-(C1-Pad2) -> unconnected-(CN1-Pad2)
- CN1 pad 3: GND -> Net-(C4-Pad2)
- CN1 pad 4: Net-(C4-Pad2) -> Net-(C1-Pad2)
- CN1 pad 5: unconnected-(CN1-Pad5) -> GND
Routing:
- net Net-(C4-Pad2): track 18.3 -> 22.3 mm, vias 1 -> 2
- net GND: track 91.8 -> 88.2 mm, vias 8 -> 7
- net Net-(C1-Pad2): track 10.6 -> 8.22 mm
