File: kicad/Audio Jack.kicad_sch (KiCad schematic)
At the start: 14 parts, among them CN1 PJ-320A, SW1 SW_Push, SW2 SW_Push, SW3 SW_Push, U1 TLV320DAC3100IRHBR

Commit message: Add files via upload
Connections:
- net GND: now also CN1.5; no longer CN1.3
- net at CN1.2: no longer C1.2
- net at C4.2: now also CN1.3; no longer CN1.4
- new net: C1.2, CN1.4
Changed lines of the file:
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@@
 	)
 	(no_connect
-		(at 163.83 48.26)
+		(at 171.45 48.26)
 	)
 	(no_connect
@@
 	(wire
 		(pts
+			(xy 163.83 48.26) (xy 163.83 44.45)
+		)
+		(stroke
+			(width 0)
+			(type default)
+		)
+	)
+	(wire
+		(pts
 			(xy 133.35 93.98) (xy 134.62 93.98)
 		)
@@
 	(wire
 		(pts
-			(xy 166.37 44.45) (xy 158.75 44.45)
-		)
-		(stroke
-			(width 0)
-			(type default)
-		)
-	)
-	(wire
-		(pts
 			(xy 106.68 113.03) (xy 106.68 111.76)
 		)
@@
 	(wire
 		(pts
-			(xy 158.75 40.64) (xy 168.91 40.64)
-		)
-		(stroke
-			(width 0)
-			(type default)
-		)
-	)
-	(wire
-		(pts
 			(xy 172.72 72.39) (xy 172.72 74.93)
 		)
@@
 	(wire
 		(pts
+			(xy 163.83 44.45) (xy 158.75 44.45)
+		)
+		(stroke
+			(width 0)
+			(type default)
+		)
+	)
+	(wire
+		(pts
 			(xy 137.16 128.27) (xy 137.16 130.81)
 		)
@@
 	(wire
 		(pts
-			(xy 171.45 40.64) (xy 198.12 40.64)
+			(xy 168.91 40.64) (xy 168.91 48.26)
 		)
 		(stroke
@@
 	(wire
 		(pts
+			(xy 158.75 40.64) (xy 166.37 40.64)
+		)
+		(stroke
+			(width 0)
+			(type default)
+		)
+	)
+	(wire
+		(pts
 			(xy 96.52 96.52) (xy 100.33 96.52)
 		)
@@
 	(wire
 		(pts
-			(xy 168.91 40.64) (xy 168.91 48.26)
-		)
-		(stroke
-			(width 0)
-			(type default)
-		)
-	)
-	(wire
-		(pts
 			(xy 139.7 116.84) (xy 139.7 115.57)
 		)
@@
 	(wire
 		(pts
+			(xy 168.91 40.64) (xy 198.12 40.64)
+		)
+		(stroke
+			(width 0)
+			(type default)
+		)
+	)
+	(wire
+		(pts
 			(xy 175.26 78.74) (xy 175.26 77.47)
 		)
@@
 	(wire
 		(pts
-			(xy 171.45 48.26) (xy 171.45 40.64)
-		)
-		(stroke
-			(width 0)
-			(type default)
-		)
-	)
-	(wire
-		(pts
 			(xy 143.51 106.68) (xy 149.86 106.68)
 		)
@@
 	(wire
 		(pts
-			(xy 166.37 48.26) (xy 166.37 44.45)
-		)
-		(stroke
-			(width 0)
-			(type default)
-		)
-	)
-	(wire
-		(pts
 			(xy 96.52 96.52) (xy 96.52 95.25)
 		)
@@
 		)
 		(stroke
+			(width 0)
+			(type default)
+		)
+	)
+	(wire
+		(pts
+			(xy 166.37 40.64) (xy 166.37 48.26)
+		)
+		(stroke
